Commit message: Cinematico a 3 braccia

File: src/simulator_2link_planar/urdf/2link_planar_model.urdf (robot description, URDF)
Before this commit: robot simple_model, 3 links, 2 joints
Links:
- added link ultimoarm_link, mass 1; visual cylinder length=1.0 radius=0.05
Joints:
- added joint ultimoarm_joint: type continuous, parent forearm_link, child ultimoarm_link, origin xyz=1.0 0 0, axis 0 0 1

Commit message: nuovo urdf non va

File: src/simulator_2link_planar/urdf/2link_planar_model.urdf (robot description, URDF)
Before this commit: robot simple_model, 4 links, 3 joints
Links:
- removed link arm_link
- removed link forearm_link
- removed link ultimoarm_link
- added link link_1, mass 0.0785942338762368; collision mesh filename=package://simulator_2link_planar/meshes/link_1.STL; visual mesh filename=package://simulator_2link_planar/meshes/link_1.STL
- added link link_2, mass 0.0785942338762368; collision mesh filename=package://simulator_2link_planar/meshes/link_2.STL; visual mesh filename=package://simulator_2link_planar/meshes/link_2.STL
- added link link_3, mass 0.0785942338762368; collision mesh filename=package://simulator_2link_planar/meshes/link_3.STL; visual mesh filename=package://simulator_2link_planar/meshes/link_3.STL
- added link link_4, mass 0.0785942338762368; collision mesh filename=package://simulator_2link_planar/meshes/link_4.STL; visual mesh filename=package://simulator_2link_planar/meshes/link_4.STL
- added link link_5, mass 0.0785942338762368; collision mesh filename=package://simulator_2link_planar/meshes/link_5.STL; visual mesh filename=package://simulator_2link_planar/meshes/link_5.STL
- added link link_6, mass 0.0279702497322662; collision mesh filename=package://simulator_2link_planar/meshes/link_6.STL; visual mesh filename=package://simulator_2link_planar/meshes/link_6.STL
- link base_link: mass None -> 0.0785942338762368; geometry collision mesh filename=package://simulator_2link_planar/meshes/base_link.STL; visual mesh filename=package://simulator_2link_planar/meshes/base_link.STL
Joints:
- removed joint arm_joint
- removed joint forearm_joint
- removed joint ultimoarm_joint
- added joint joint_1: type continuous, parent base_link, child link_1, origin xyz=0.057188 0.0059831 0.13343 rpy=1.5708 6.9389E-16 -3.1416, axis 0 1 0
- added joint joint_2: type continuous, parent link_1, child link_2, origin xyz=0 0.18967 0 rpy=0.94237 -0.4634 -0.11653, axis -0.88847 0.2908 0.35504
- added joint joint_3: type continuous, parent link_2, child link_3, origin xyz=-0.024558 0.12737 -0.16578 rpy=0.97336 -0.36296 2.8253, axis 1 0 0
- added joint joint_4: type fixed, parent link_3, child link_4, origin xyz=0.0088 -0.1588 0 rpy=-1.5708 0 0, axis 0 0 -1
- added joint joint_5: type fixed, parent link_4, child link_5, origin xyz=0 0 -0.1053 rpy=3.1416 1.1102E-14 3.1416, axis -1 0 0
- added joint joint_6: type fixed, parent link_5, child link_6, origin xyz=-0.0039 0 0.1636 rpy=-1.5708 1.249E-14 0, axis 0 -1 0
