Commit message: Matlab per dinamico a 3

File: urdf/2link_planar_model.urdf (robot description, URDF)
Before this commit: robot edo_sim, 7 links, 6 joints
Joints:
- joint joint_4: type continuous -> fixed
- joint joint_5: type continuous -> fixed
- joint joint_6: type continuous -> fixed

Commit message: Corrette inerzie urdf

File: urdf/2link_planar_model.urdf (robot description, URDF)
Before this commit: robot edo_sim, 7 links, 6 joints
Links:
- link base_link: mass 0.0785942338762368 -> 7.49
- link link_1: mass 0.0785942338762368 -> 2.071768
- link link_2: mass 0.0785942338762368 -> 1.333978
- link link_3: mass 0.0785942338762368 -> 6.22909E-01
- link link_4: mass 0.0785942338762368 -> 5.2005E-01
- link link_5: mass 0.0785942338762368 -> 5.41662E-01
- link link_6: mass 0.0279702497322662 -> 9.5445E-02
