Commit message: Sbloccati ultimi joint

File: src/edo/urdf/edo.xacro (robot description, xacro)
@@ -154,5 +154,5 @@
             </collision>
         </link>
-        <joint name="${robot_prefix}_joint_4" type="fixed">
+        <joint name="${robot_prefix}_joint_4" type="revolute">
             <parent link="${robot_prefix}_link_3"/>
             <child link="${robot_prefix}_link_4"/>
@@ -190,5 +190,5 @@
             </collision>
         </link>
-        <joint name="${robot_prefix}_joint_5" type="fixed">
+        <joint name="${robot_prefix}_joint_5" type="revolute">
             <parent link="${robot_prefix}_link_4"/>
             <child link="${robot_prefix}_link_5"/>
@@ -226,5 +226,5 @@
             </collision>
         </link>
-        <joint name="${robot_prefix}_joint_6" type="fixed">
+        <joint name="${robot_prefix}_joint_6" type="revolute">
             <parent link="${robot_prefix}_link_5"/>
             <child link="${robot_prefix}_link_6"/>
